Commit message: Update turtlebot3_waffle_pi_with_box.urdf

File: turtlebot3_description_ros1/urdf/turtlebot3_waffle_pi_with_box.urdf (robot description, URDF)
Before this commit: robot turtlebot3_waffle_pi, 28 links, 27 joints
Links:
- link stand_fl: mass 0.01 -> 0.1; geometry collision box size=0.003 0.003 0.45; visual box size=0.003 0.003 0.45
- link stand_fr: mass 0.01 -> 0.1; geometry collision box size=0.003 0.003 0.45; visual box size=0.003 0.003 0.45
- link stand_rl: mass 0.01 -> 0.1; geometry collision box size=0.003 0.003 0.45; visual box size=0.003 0.003 0.45
- link stand_rr: mass 0.01 -> 0.1; geometry collision box size=0.003 0.003 0.45; visual box size=0.003 0.003 0.45
Joints:
- joint base_standfl_joint: origin xyz=0.05 -0.1 0.35 rpy=0 0 0 -> xyz=0.05 -0.1 0.315 rpy=0 0 0
- joint base_standfr_joint: origin xyz=0.05 0.1 0.35 rpy=0 0 0 -> xyz=0.05 0.1 0.315 rpy=0 0 0
- joint base_standrl_joint: origin xyz=-0.15 0.1 0.35 rpy=0 0 0 -> xyz=-0.18 0.1 0.315 rpy=0 0 0
- joint base_standrr_joint: origin xyz=-0.15 -0.1 0.35 rpy=0 0 0 -> xyz=-0.18 -0.1 0.315 rpy=0 0 0
- joint stand_plate_joint: origin xyz=-0.05 -0.1 0.15 rpy=0 0 1.57 -> xyz=-0.1 -0.1 0.225 rpy=0 0 1.57
